Commit message: changes

File: aliengo_description/xacro/robot.xacro (robot description, xacro)
@@ -178,12 +178,12 @@
             <origin rpy="0 0 0" xyz="0 0 0"/>
             <geometry>
-                       <mesh filename="package://aliengo_description/xacro/belt.stl" scale="0.1 0.3 0.1"/>
-            </geometry>
-            <material name="red"/>
-        </visual>
-        <collision>
-            <origin rpy="0 0 0" xyz="0 0 0"/>
-            <geometry>
-                <mesh filename="package://aliengo_description/xacro/belt.stl" scale="0.1 0.3 0.1"/>
+                       <mesh filename="package://aliengo_description/xacro/belt.stl" scale="0.05 0.3 0.1"/>
+            </geometry>
+            <material name="red"/>
+        </visual>
+        <collision>
+            <origin rpy="0 0 0" xyz="0 0 0"/>
+            <geometry>
+                <mesh filename="package://aliengo_description/xacro/belt.stl" scale="0.05 0.3 0.1"/>
             </geometry>
         </collision>

Commit message: stable

File: aliengo_description/xacro/robot.xacro (robot description, xacro)
@@ -167,9 +167,9 @@
         <parent link="trunk"/>
         <child link="aliengo_belt_link"/>
-        <origin rpy="0 0 1.54" xyz="0 0 0.2"/>
+        <origin rpy="0 0 0" xyz="0 0 0.1"/>
     </joint>
      <link name="aliengo_belt_link">
         <inertial>
-            <mass value="0.0001"/>
+            <mass value="0.01"/>
             <origin rpy="0 0 0" xyz="0 0 0"/>
             <inertia ixx="0.0001" ixy="0" ixz="0" iyy="0.0001" iyz="0" izz="0.0001"/>
@@ -178,12 +178,12 @@
             <origin rpy="0 0 0" xyz="0 0 0"/>
             <geometry>
-                       <mesh filename="package://aliengo_description/xacro/belt.stl" scale="0.05 0.3 0.1"/>
-            </geometry>
-            <material name="red"/>
-        </visual>
-        <collision>
-            <origin rpy="0 0 0" xyz="0 0 0"/>
-            <geometry>
-                <mesh filename="package://aliengo_description/xacro/belt.stl" scale="0.05 0.3 0.1"/>
+                       <mesh filename="package://aliengo_description/xacro/aliengo_deck.stl" scale="1 1 1"/>
+            </geometry>
+            <material name="red"/>
+        </visual>
+        <collision>
+            <origin rpy="0 0 0" xyz="0 0 0"/>
+            <geometry>
+                <mesh filename="package://aliengo_description/xacro/aliengo_deck.stl" scale="1 1 1"/>
             </geometry>
         </collision>
